File: SparkFun-Wearable-Shield-For-Photon.brd (EAGLE design)
At the start: 59.7 x 59.7 mm, 54 parts, among them J1 PAD, J10 PAD, J11 PAD, J12 PAD, J13 PAD, J14 PAD, J15 PAD, J16 PAD, J17 PAD, J18 PAD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

Commit message: Updating Boards
Parts:
- removed U$1: (no value), SparkFun-Aesthetics:OSHW-LOGO-M
- removed U$2: (no value), SparkFun-Aesthetics:SFE_LOGO_FLAME_.2
- added FID1, FID2: FIDUCIAL1X2, SparkFun-Aesthetics:FIDUCIAL-1X2
- added LOGO1: SFE_LOGO_FLAME.2_INCH, SparkFun-Aesthetics:SFE_LOGO_FLAME_.2
- added LOGO2: OSHW-LOGOM, SparkFun-Aesthetics:OSHW-LOGO-M
Connections:
- removed net VCC: JP1.1
- net VIN: now also JP1.1
Routing:
- net D0: track 32.7 -> 28.0 mm
Other:
- board text added: "V01"
- board text added: "Wearable Breakout For Photon"
- board text removed: "Photon Wearables Breakout"
- board text removed: "REV10"
- board text removed: "Tips for using the SparkFun Photon Wearables Breakout: - Use conductive thread with the larger pin holes. - Solder wires with the smaller pin holes. - Use conductive paint or copper tape with the larger pin holes. ~ Happy Hacking"
Changed lines of the file:
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@@
 <drawing>
 <settings>
-<setting alwaysvectorfont="no"/>
+<setting alwaysvectorfont="yes"/>
 <setting verticaltext="up"/>
 </settings>
@@
 <layer number="27" name="tValues" color="7" fill="1" visible="no" active="yes"/>
 <layer number="28" name="bValues" color="7" fill="1" visible="no" active="yes"/>
-<layer number="29" name="tStop" color="7" fill="3" visible="yes" active="yes"/>
-<layer number="30" name="bStop" color="7" fill="6" visible="yes" active="yes"/>
+<layer number="29" name="tStop" color="7" fill="3" visible="no" active="yes"/>
+<layer number="30" name="bStop" color="7" fill="6" visible="no" active="yes"/>
 <layer number="31" name="tCream" color="7" fill="4" visible="no" active="yes"/>
 <layer number="32" name="bCream" color="7" fill="5" visible="no" active="yes"/>
@@
 <layer number="45" name="Holes" color="7" fill="1" visible="yes" active="yes"/>
 <layer number="46" name="Milling" color="3" fill="1" visible="no" active="yes"/>
-<layer number="47" name="Measures" color="7" fill="1" visible="no" active="yes"/>
+<layer number="47" name="Measures" color="7" fill="1" visible="yes" active="yes"/>
 <layer number="48" name="Document" color="7" fill="1" visible="no" active="yes"/>
-<layer number="49" name="Reference" color="7" fill="1" visible="no" active="yes"/>
+<layer number="49" name="Reference" color="7" fill="1" visible="yes" active="yes"/>
 <layer number="50" name="dxf" color="7" fill="1" visible="no" active="no"/>
 <layer number="51" name="tDocu" color="6" fill="1" visible="yes" active="yes"/>
-<layer number="52" name="bDocu" color="7" fill="1" visible="yes" active="yes"/>
+<layer number="52" name="bDocu" color="7" fill="1" visible="no" active="yes"/>
 <layer number="53" name="tGND_GNDA" color="7" fill="1" visible="no" active="no"/>
 <layer number="54" name="bGND_GNDA" color="7" fill="1" visible="no" active="no"/>
@@
 <board>
 <plain>
-<circle x="29.726128125" y="30.110428125" radius="29.845" width="0.254" layer="20"/>
+<circle x="29.726128125" y="30.110428125" radius="29.845" width="0.2032" layer="20"/>
 <wire x1="19.566128125" y1="44.810425" x2="19.566128125" y2="47.890428125" width="0.254" layer="21"/>
 <wire x1="19.566128125" y1="47.890428125" x2="39.886128125" y2="47.890428125" width="0.254" layer="21"/>
@@
 <text x="13.88465625" y="39.330628125" size="1.27" layer="21" ratio="15" align="center">WKP</text>
 <text x="12.083034375" y="35.0527625" size="1.27" layer="21" ratio="15" align="center">DAC</text>
-<text x="10.69975" y="30.1284625" size="1.27" layer="21" ratio="15" align="center">A5</text>
-<text x="11.501628125" y="25.092403125" size="1.27" layer="21" ratio="15" align="center">A4</text>
+<text x="10.69975" y="30.1284625" size="1.27" layer="21" font="vector" ratio="15" align="center">A5</text>
+<text x="11.501628125" y="25.092403125" size="1.27" layer="21" font="vector" ratio="15" align="center">A4</text>
 <text x="13.29258125" y="20.5425" size="1.27" layer="21" ratio="15" align="center">A3</text>
 <text x="16.521684375" y="16.4665625" size="1.27" layer="21" ratio="15" align="center">A2</text>
@@
 <text x="42.172384375" y="47.151540625" size="1.27" layer="21" ratio="15" rot="R180" align="center">RST</text>
 <text x="34.917384375" y="49.214528125" size="1.27" layer="21" ratio="15" rot="R180" align="center">3V3</text>
-<text x="29.7782" y="28.354015625" size="1.27" layer="21" ratio="15" align="center">Photon
-Wearables
-Breakout</text>
+<text x="29.7782" y="28.354015625" size="1.27" layer="21" ratio="15" align="center">Wearable
+Breakout
+For Photon</text>
 <wire x1="89.416128125" y1="13.600428125" x2="88.146128125" y2="11.060428125" width="0.254" layer="106"/>
 <text x="29.747209375" y="49.979834375" size="1.27" layer="22" ratio="15" rot="MR0" align="center">VIN</text>
@@
 <text x="41.93641875" y="47.3577875" size="1.27" layer="22" ratio="15" rot="MR180" align="center">RST</text>
 <text x="34.917384375" y="49.214528125" size="1.27" layer="22" ratio="15" rot="MR180" align="center">3V3</text>
-<text x="38.22649375" y="28.5932875" size="1.016" layer="22" ratio="15" rot="MR0" align="center-left">Tips for using the
-SparkFun Photon
-Wearables Breakout:
-- Use conductive thread
-with the larger pin holes.
-- Solder wires with the
-smaller pin holes.
-- Use conductive paint or
-copper tape with the larger
-pin holes.
-~ Happy Hacking
-</text>
 <text x="27.803346875" y="-13.970253125" size="1.778" layer="51">Pamela Cortez</text>
-<text x="32.283909375" y="16.523715625" size="1.27" layer="16" font="vector" ratio="15" rot="MR0">REV10</text>
+<text x="31.013909375" y="19.063715625" size="1.27" layer="16" font="vector" ratio="15" rot="MR0">V01</text>
+<dimension x1="-0.118859375" y1="30.13925625" x2="59.571115625" y2="30.0816" x3="29.756096875" y3="61.138815625" textsize="1.778" layer="47" dtype="diameter" unit="inch"/>
 </plain>
 <attributes>
@@
 <element name="JP14" library="SparkFun-Connectors" package="1X01NS" value="M01SMDNS" x="40.724328125" y="49.160428125" rot="R240"/>
 <element name="JP13" library="SparkFun-Connectors" package="1X01NS" value="M01SMDNS" x="35.415728125" y="51.370228125" rot="R255"/>
-<element name="U$1" library="SparkFun-Aesthetics" package="OSHW-LOGO-M" value="" x="44.66793125" y="30.34486875"/>
-<element name="U$2" library="SparkFun-Aesthetics" package="SFE_LOGO_FLAME_.2" value="" x="13.01623125" y="27.64205625"/>
 <element name="U$3" library="SparkFun-Aesthetics" package="SFE_LOGO_NAME_.1" value="" x="23.8196125" y="30.93770625"/>
+<element name="LOGO1" library="SparkFun-Aesthetics" package="SFE_LOGO_FLAME_.2" value="SFE_LOGO_FLAME.2_INCH" x="13.407390625" y="27.62605625"/>
+<element name="LOGO2" library="SparkFun-Aesthetics" package="OSHW-LOGO-M" value="OSHW-LOGOM" x="44.63415" y="30.16834375"/>
+<element name="FID1" library="SparkFun-Aesthetics" package="FIDUCIAL-1X2" value="FIDUCIAL1X2" x="38.018971875" y="50.490375"/>
+<element name="FID2" library="SparkFun-Aesthetics" package="FIDUCIAL-1X2" value="FIDUCIAL1X2" x="12.346178125" y="17.2648875"/>
 </elements>
 <signals>
@@
 <wire x1="29.726128125" y1="8.088628125" x2="29.726128125" y2="3.470428125" width="0.254" layer="1"/>
 <wire x1="36.966128125" y1="16.140428125" x2="40.266128125" y2="16.140428125" width="0.4064" layer="1"/>
-<wire x1="26.67" y1="11.14475625" x2="26.67" y2="19.05" width="0.254" layer="1"/>
-<wire x1="26.67" y1="19.05" x2="27.94" y2="20.32" width="0.254" layer="1"/>
-<wire x1="27.94" y1="20.32" x2="31.75" y2="20.32" width="0.254" layer="1"/>
-<wire x1="31.75" y1="20.32" x2="35.929571875" y2="16.140428125" width="0.254" layer="1"/>
+<wire x1="26.67" y1="11.14475625" x2="26.67" y2="15.24" width="0.254" layer="1"/>
+<wire x1="28.324046875" y1="16.14119375" x2="31.570675" y2="16.141190625" width="0.254" layer="1"/>
 <wire x1="35.929571875" y1="16.140428125" x2="36.966128125" y2="16.140428125" width="0.254" layer="1"/>
 <wire x1="29.726128125" y1="8.088628125" x2="26.67" y2="11.14475625" width="0.254" layer="1"/>
+<wire x1="31.570675" y1="16.141190625" x2="33.389571875" y2="16.140428125" width="0.254" layer="1"/>
+<wire x1="33.389571875" y1="16.140428125" x2="36.966128125" y2="16.140428125" width="0.254" layer="1"/>
+<wire x1="26.67" y1="15.24" x2="27.57119375" y2="16.14119375" width="0.254" layer="1"/>
+<wire x1="27.57119375" y1="16.14119375" x2="28.324046875" y2="16.14119375" width="0.254" layer="1"/>
 </signal>
 <signal name="VIN">
@@
 <wire x1="29.726128125" y1="45.350428125" x2="28.456128125" y2="44.080428125" width="0.254" layer="1"/>
 <wire x1="28.456128125" y1="44.080428125" x2="22.486128125" y2="44.080428125" width="0.254" layer="1"/>
-<wire x1="29.726128125" y1="56.750428125" x2="29.726128125" y2="45.350428125" width="0.254" layer="1"/>
+<contactref element="JP1" pad="1"/>
+<wire x1="29.726128125" y1="56.750428125" x2="29.726128125" y2="52.132240625" width="0.254" layer="1"/>
+<wire x1="29.726128125" y1="52.132240625" x2="29.726128125" y2="45.350428125" width="0.254" layer="1"/>
 </signal>
 <signal name="GND">
@@
 <wire x1="22.486128125" y1="16.140428125" x2="23.376128125" y2="16.140428125" width="0.254" layer="1"/>
 </signal>
-<signal name="VCC">
-<contactref element="JP1" pad="1"/>
-</signal>
 </signals>
