File: SparkFun-Photon-Wearable-Shield.brd (EAGLE design)
At the start: 59.7 x 59.7 mm, 56 parts, among them J1 PAD, J10 PAD, J11 PAD, J12 PAD, J13 PAD, J14 PAD, J15 PAD, J16 PAD, J17 PAD, J18 PAD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

Commit message: Updating board files
V10
Parts:
- removed U$3: (no value), SparkFun-Aesthetics:SFE_LOGO_NAME_.1
- added LOGO3: SFE_LOGO_NAME_FLAME.1_INCH, SparkFun-Aesthetics:SFE_LOGO_NAME_FLAME_.1
- added U$2: (no value), SparkFun-Aesthetics:SFE_LOGO_FLAME_.9
Other:
- board text added: "Photon Wearable Shield"
- board text added: "V10"
- board text removed: "V01"
- board text removed: "Wearable Breakout For Photon"
