File: SparkFun-Photon-Wearable-Shield.sch (EAGLE design)
At the start: 55 parts, among them J1 PAD, J10 PAD, J11 PAD, J12 PAD, J13 PAD, J14 PAD, J15 PAD, J16 PAD, J17 PAD, J18 PAD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

Commit message: Updating board files
V10
Parts:
- added LOGO3: SFE_LOGO_NAME_FLAME.1_INCH, SparkFun-Aesthetics:SFE_LOGO_NAME_FLAME.1_INCH
Other:
- note added: "V10"
- note removed: "V01"
Changed lines of the file:
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@@
 <part name="FID1" library="SparkFun-Aesthetics" deviceset="FIDUCIAL" device="1X2"/>
 <part name="FID2" library="SparkFun-Aesthetics" deviceset="FIDUCIAL" device="1X2"/>
+<part name="LOGO3" library="SparkFun-Aesthetics" deviceset="SFE_LOGO_NAME_FLAME" device=".1_INCH"/>
 </parts>
 <sheets>
@@
 <plain>
 <text x="170.942" y="11.43" size="2.54" layer="94">Pamela Cortez</text>
-<text x="235.966" y="6.858" size="2.54" layer="94">V01</text>
+<text x="235.966" y="6.858" size="2.54" layer="94">V10</text>
 <wire x1="106.68" y1="185.42" x2="106.68" y2="0" width="0.1524" layer="97" style="shortdash"/>
 <text x="25.4" y="167.64" size="2.54" layer="97">0.01" Soldering Connectors
@@
 <instance part="3V3" gate="G$1" x="71.628" y="157.48"/>
 <instance part="VIN" gate="G$1" x="35.56" y="157.48"/>
-<instance part="LOGO1" gate="G$1" x="212.344" y="38.354"/>
-<instance part="LOGO2" gate="G$1" x="235.204" y="46.228"/>
+<instance part="LOGO1" gate="G$1" x="128.524" y="5.334"/>
+<instance part="LOGO2" gate="G$1" x="133.604" y="30.988"/>
 <instance part="FID1" gate="G$1" x="137.922" y="2.54"/>
 <instance part="FID2" gate="G$1" x="143.002" y="2.54"/>
+<instance part="LOGO3" gate="G$1" x="170.18" y="40.64"/>
 </instances>
 <busses>
